File: TeensyJoystick/TeensyJoystick.kicad_pcb (KiCad board)
At the start: 2 copper layers, 43.2 x 63.5 mm, 11 parts, among them J1 TEENSY3.2-72MHz, M101 THUMB_STICK, SW1 SW_Push, SW2 SW_Push, SW3 SW_Push

Commit message: Finish Teensy Joystick.
Parts:
- added R1: R, Resistors_THT:R_Axial_DIN0204_L3.6mm_D1.6mm_P7.62mm_Horizontal, F.Cu at (48.3, 100.3)
- added R2: R, Resistors_THT:R_Axial_DIN0204_L3.6mm_D1.6mm_P7.62mm_Horizontal, F.Cu at (83.8, 100.3)
Routing:
- net Net-(D2-Pad1): track 0.00 -> 2.54 mm
- net Net-(D1-Pad1): track 0.00 -> 2.54 mm
Changed lines of the file:
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@@
     (links 30)
     (no_connects 0)
-    (area 34.154533 59.3344 105.545468 133.781801)
+    (area 44.373799 63.423799 87.706201 127.076201)
     (thickness 1.6)
     (drawings 10)
-    (tracks 44)
+    (tracks 46)
     (zones 0)
-    (modules 11)
+    (modules 13)
     (nets 33)
   )
@@
     (pad 1 np_thru_hole circle (at 0 0) (size 2.7 2.7) (drill 2.7) (layers *.Cu *.Mask))
   )
+  (module Resistors_THT:R_Axial_DIN0204_L3.6mm_D1.6mm_P7.62mm_Horizontal (layer F.Cu)
+    (at 48.26 100.33 90)
+    (descr "Resistor, Axial_DIN0204 series, Axial, Horizontal, pin pitch=7.62mm, 0.16666666666666666W = 1/6W, length*diameter=3.6*1.6mm^2, http://cdn-reichelt.de/documents/datenblatt/B400/1_4W%23YAG.pdf")
+    (tags "Resistor Axial_DIN0204 series Axial Horizontal pin pitch 7.62mm 0.16666666666666666W = 1/6W length 3.6mm diameter 1.6mm")
+    (fp_text reference R1 (at 3.81 -1.86 90) (layer F.SilkS)
+      (effects (font (size 1 1) (thickness 0.15)))
+    )
+    (fp_text value R (at 3.81 1.86 90) (layer F.Fab)
+      (effects (font (size 1 1) (thickness 0.15)))
+    )
+    (fp_line (start 2.01 -0.8) (end 2.01 0.8) (layer F.Fab) (width 0.1))
+    (fp_line (start 2.01 0.8) (end 5.61 0.8) (layer F.Fab) (width 0.1))
+    (fp_line (start 5.61 0.8) (end 5.61 -0.8) (layer F.Fab) (width 0.1))
+    (fp_line (start 5.61 -0.8) (end 2.01 -0.8) (layer F.Fab) (width 0.1))
+    (fp_line (start 0 0) (end 2.01 0) (layer F.Fab) (width 0.1))
+    (fp_line (start 7.62 0) (end 5.61 0) (layer F.Fab) (width 0.1))
+    (fp_line (start 1.95 -0.86) (end 1.95 0.86) (layer F.SilkS) (width 0.12))
+    (fp_line (start 1.95 0.86) (end 5.67 0.86) (layer F.SilkS) (width 0.12))
+    (fp_line (start 5.67 0.86) (end 5.67 -0.86) (layer F.SilkS) (width 0.12))
+    (fp_line (start 5.67 -0.86) (end 1.95 -0.86) (layer F.SilkS) (width 0.12))
+    (fp_line (start 0.88 0) (end 1.95 0) (layer F.SilkS) (width 0.12))
+    (fp_line (start 6.74 0) (end 5.67 0) (layer F.SilkS) (width 0.12))
+    (fp_line (start -0.95 -1.15) (end -0.95 1.15) (layer F.CrtYd) (width 0.05))
+    (fp_line (start -0.95 1.15) (end 8.6 1.15) (layer F.CrtYd) (width 0.05))
+    (fp_line (start 8.6 1.15) (end 8.6 -1.15) (layer F.CrtYd) (width 0.05))
+    (fp_line (start 8.6 -1.15) (end -0.95 -1.15) (layer F.CrtYd) (width 0.05))
+    (pad 1 thru_hole circle (at 0 0 90) (size 1.4 1.4) (drill 0.7) (layers *.Cu *.Mask)
+      (net 3 GND))
+    (pad 2 thru_hole oval (at 7.62 0 90) (size 1.4 1.4) (drill 0.7) (layers *.Cu *.Mask)
+      (net 4 "Net-(D1-Pad1)"))
+    (model ${KISYS3DMOD}/Resistors_THT.3dshapes/R_Axial_DIN0204_L3.6mm_D1.6mm_P7.62mm_Horizontal.wrl
+      (at (xyz 0 0 0))
+      (scale (xyz 0.393701 0.393701 0.393701))
+      (rotate (xyz 0 0 0))
+    )
+  )
+  (module Resistors_THT:R_Axial_DIN0204_L3.6mm_D1.6mm_P7.62mm_Horizontal (layer F.Cu)
+    (at 83.82 100.33 90)
+    (descr "Resistor, Axial_DIN0204 series, Axial, Horizontal, pin pitch=7.62mm, 0.16666666666666666W = 1/6W, length*diameter=3.6*1.6mm^2, http://cdn-reichelt.de/documents/datenblatt/B400/1_4W%23YAG.pdf")
+    (tags "Resistor Axial_DIN0204 series Axial Horizontal pin pitch 7.62mm 0.16666666666666666W = 1/6W length 3.6mm diameter 1.6mm")
+    (fp_text reference R2 (at 3.81 -1.86 90) (layer F.SilkS)
+      (effects (font (size 1 1) (thickness 0.15)))
+    )
+    (fp_text value R (at 3.81 1.86 90) (layer F.Fab)
+      (effects (font (size 1 1) (thickness 0.15)))
+    )
+    (fp_line (start 2.01 -0.8) (end 2.01 0.8) (layer F.Fab) (width 0.1))
+    (fp_line (start 2.01 0.8) (end 5.61 0.8) (layer F.Fab) (width 0.1))
+    (fp_line (start 5.61 0.8) (end 5.61 -0.8) (layer F.Fab) (width 0.1))
+    (fp_line (start 5.61 -0.8) (end 2.01 -0.8) (layer F.Fab) (width 0.1))
+    (fp_line (start 0 0) (end 2.01 0) (layer F.Fab) (width 0.1))
+    (fp_line (start 7.62 0) (end 5.61 0) (layer F.Fab) (width 0.1))
+    (fp_line (start 1.95 -0.86) (end 1.95 0.86) (layer F.SilkS) (width 0.12))
+    (fp_line (start 1.95 0.86) (end 5.67 0.86) (layer F.SilkS) (width 0.12))
+    (fp_line (start 5.67 0.86) (end 5.67 -0.86) (layer F.SilkS) (width 0.12))
+    (fp_line (start 5.67 -0.86) (end 1.95 -0.86) (layer F.SilkS) (width 0.12))
+    (fp_line (start 0.88 0) (end 1.95 0) (layer F.SilkS) (width 0.12))
+    (fp_line (start 6.74 0) (end 5.67 0) (layer F.SilkS) (width 0.12))
+    (fp_line (start -0.95 -1.15) (end -0.95 1.15) (layer F.CrtYd) (width 0.05))
+    (fp_line (start -0.95 1.15) (end 8.6 1.15) (layer F.CrtYd) (width 0.05))
+    (fp_line (start 8.6 1.15) (end 8.6 -1.15) (layer F.CrtYd) (width 0.05))
+    (fp_line (start 8.6 -1.15) (end -0.95 -1.15) (layer F.CrtYd) (width 0.05))
+    (pad 1 thru_hole circle (at 0 0 90) (size 1.4 1.4) (drill 0.7) (layers *.Cu *.Mask)
+      (net 3 GND))
+    (pad 2 thru_hole oval (at 7.62 0 90) (size 1.4 1.4) (drill 0.7) (layers *.Cu *.Mask)
+      (net 6 "Net-(D2-Pad1)"))
+    (model ${KISYS3DMOD}/Resistors_THT.3dshapes/R_Axial_DIN0204_L3.6mm_D1.6mm_P7.62mm_Horizontal.wrl
+      (at (xyz 0 0 0))
+      (scale (xyz 0.393701 0.393701 0.393701))
+      (rotate (xyz 0 0 0))
+    )
+  )
   (dimension 58.42 (width 0.1524) (layer Cmts.User)
     (gr_text "58.420 mm" (at 38.5572 95.25 270) (layer Cmts.User)
@@
   (via (at 66.04 71.12) (size 0.6858) (drill 0.3302) (layers F.Cu B.Cu) (net 2))
   (segment (start 64.77 90.17) (end 64.77 86.36) (width 0.254) (layer F.Cu) (net 2))
+  (segment (start 48.26 90.17) (end 48.26 92.71) (width 0.254) (layer F.Cu) (net 4))
   (segment (start 74.93 87.63) (end 74.93 84.51799) (width 0.254) (layer F.Cu) (net 5))
   (segment (start 74.93 84.51799) (end 74.93 83.82) (width 0.254) (layer F.Cu) (net 5))
   (segment (start 48.26 87.63) (end 74.93 87.63) (width 0.254) (layer B.Cu) (net 5))
   (via (at 74.93 87.63) (size 0.6858) (drill 0.3302) (layers F.Cu B.Cu) (net 5))
+  (segment (start 83.82 90.17) (end 83.82 92.71) (width 0.254) (layer F.Cu) (net 6))
   (segment (start 77.47 87.63) (end 83.82 87.63) (width 0.254) (layer B.Cu) (net 7))
   (segment (start 77.47 83.82) (end 77.47 87.63) (width 0.254) (layer F.Cu) (net 7))
@@
     (connect_pads (clearance 0.508))
     (min_thickness 0.254)
-    (fill (arc_segments 16) (thermal_gap 0.508) (thermal_bridge_width 0.508))
+    (fill yes (arc_segments 16) (thermal_gap 0.508) (thermal_bridge_width 0.508))
     (polygon
       (pts
@@
     (connect_pads (clearance 0.508))
     (min_thickness 0.254)
-    (fill (arc_segments 16) (thermal_gap 0.508) (thermal_bridge_width 0.508))
+    (fill yes (arc_segments 16) (thermal_gap 0.508) (thermal_bridge_width 0.508))
     (polygon
       (pts
