File: DCDC3_7-5+12/DCDC3-7-5.sch (KiCad schematic (older format))
At the start: 7 parts, among them U2 XL6009

Commit message: Final version of aux 5v and 12v power supply.
Parts:
- L2: Mouser Part Number (none) -> 542-PM5022S-330M-RC
- R3: Mouser Part Number (none) -> 71-CRCW0805-3K
- R4: Mouser Part Number (none) -> 71-CRCW08051K00FKEAH
- U2: XLSEMI Part Number (none) -> XL6009
Changed lines of the file:
@@
 F 2 "TO_SOT_Packages_SMD:TO-263-5_TabPin3" H 5600 3700 60  0001 C CNN
 F 3 "" H 5600 3700 60  0001 C CNN
+F 4 "XL6009" H 5600 3700 60  0001 C CNN "XLSEMI Part Number"
 	1    5600 3700
 	-1   0    0    -1
@@
 F 2 "PM5022S-330M-RC:INDPM183140X690N" H 5150 2800 50  0001 C CNN
 F 3 "" H 5150 2800 50  0001 C CNN
+F 4 "542-PM5022S-330M-RC" H 5150 2800 60  0001 C CNN "Mouser Part Number"
 	1    5150 2800
 	0    -1   -1   0
@@
 F 2 "Resistors_SMD:R_0805_HandSoldering" V 6180 3150 50  0001 C CNN
 F 3 "" H 6250 3150 50  0001 C CNN
+F 4 "71-CRCW0805-3K" V 6250 3150 60  0001 C CNN "Mouser Part Number"
 	1    6250 3150
 	1    0    0    -1
@@
 F 2 "Resistors_SMD:R_0805_HandSoldering" V 6180 3750 50  0001 C CNN
 F 3 "" H 6250 3750 50  0001 C CNN
+F 4 "71-CRCW08051K00FKEAH" V 6250 3750 60  0001 C CNN "Mouser Part Number"
 	1    6250 3750
 	1    0    0    -1

Commit message: Final version of aux 5v and 12v power supply.
Parts:
- U2: Manufacturer (none) -> XLSEMI; Mfg Part # (none) -> XL6009
Changed lines of the file:
@@
 F 3 "" H 5600 3700 60  0001 C CNN
 F 4 "XL6009" H 5600 3700 60  0001 C CNN "XLSEMI Part Number"
+F 5 "XLSEMI" H 5600 3700 60  0001 C CNN "Manufacturer"
+F 6 "XL6009" H 5600 3700 60  0001 C CNN "Mfg Part #"
 	1    5600 3700
 	-1   0    0    -1
